Commit message: Add UFactory 6-axis F/T sensor (AI1302) to xArm description
Introduces an optional mounting-adapter + sensor-body link pair that
splices between link<dof> and link_eef when add_ft_sensor is true, so
all downstream tool macros (gripper / vacuum / bio / other_geometry)
continue to attach at link_eef without modification.

Geometry: 30 mm adapter plate (OD 80 mm, cylinder primitive) + 61 mm
sensor body (mesh of UFactory AI1302, OD ~75 mm). Mass split 140 g /
305 g of the datasheet's 445 g total. The wrench reference frame
link_ft_sensor sits at the tool-output face, +Z toward the tool.

Defaults for add_gripper and add_ft_sensor are flipped to true to
match the TorqueAGI xArm6 build (xArm Gripper + FT sensor permanently
installed). Set either arg to false at launch time to opt out.

File: xarm_description/urdf/xarm_device.urdf.xacro (robot description, xacro)
@@ -6,7 +6,8 @@
   <xacro:arg name="effort_control" default="false"/>
   <xacro:arg name="velocity_control" default="false"/>
-  <xacro:arg name="add_gripper" default="false"/>
+  <xacro:arg name="add_gripper" default="true"/>
   <xacro:arg name="add_vacuum_gripper" default="false"/>
   <xacro:arg name="add_bio_gripper" default="false"/>
+  <xacro:arg name="add_ft_sensor" default="true"/>
   <xacro:arg name="model1300" default="false"/>
   <xacro:arg name="dof" default="7"/>
@@ -44,5 +45,5 @@
     effort_control="$(arg effort_control)" velocity_control="$(arg velocity_control)"
     add_gripper="$(arg add_gripper)" add_vacuum_gripper="$(arg add_vacuum_gripper)"
-    add_bio_gripper="$(arg add_bio_gripper)" dof="$(arg dof)"
+    add_bio_gripper="$(arg add_bio_gripper)" add_ft_sensor="$(arg add_ft_sensor)" dof="$(arg dof)"
     ros2_control_plugin="$(arg ros2_control_plugin)" robot_type="$(arg robot_type)"
     load_gazebo_plugin="true" ros2_control_params="$(arg ros2_control_params)"

File: xarm_description/urdf/xarm_device_macro.xacro (robot description, xacro)
@@ -7,7 +7,8 @@
     effort_control:=false
     velocity_control:=false
-    add_gripper:=false
+    add_gripper:=true
     add_vacuum_gripper:=false
     add_bio_gripper:=false
+    add_ft_sensor:=true
     dof:=7
     robot_type:='xarm'
@@ -218,12 +219,25 @@
       </xacro:if>
     </xacro:if>
+    <xacro:if value="${add_ft_sensor}">
+      <xacro:include filename="$(find xarm_description)/urdf/ft_sensor/xarm_ft_sensor.urdf.xacro" />
+      <xacro:xarm_ft_sensor_urdf prefix="${prefix}" attach_to="${prefix}link${dof}" />
+    </xacro:if>
     <xacro:unless value="${add_realsense_d435i}">
       <link name="${prefix}link_eef"/>
     </xacro:unless>
-    <joint name="${prefix}joint_eef" type="fixed">
-      <origin xyz="0 0 0" rpy="0 0 0" />
-      <parent link="${prefix}link${dof}" />
-      <child link="${prefix}link_eef" />
-    </joint>
+    <xacro:if value="${add_ft_sensor}">
+      <joint name="${prefix}joint_eef" type="fixed">
+        <origin xyz="0 0 0" rpy="0 0 0" />
+        <parent link="${prefix}link_ft_sensor" />
+        <child link="${prefix}link_eef" />
+      </joint>
+    </xacro:if>
+    <xacro:unless value="${add_ft_sensor}">
+      <joint name="${prefix}joint_eef" type="fixed">
+        <origin xyz="0 0 0" rpy="0 0 0" />
+        <parent link="${prefix}link${dof}" />
+        <child link="${prefix}link_eef" />
+      </joint>
+    </xacro:unless>
     <xacro:if value="${add_gripper}">
       <xacro:if value="${robot_type == 'lite'}">
