Commit message: Thread add_ft_sensor through xArm6 SRDF and MoveIt builder
Add FT joints to the xarm6 planning group and disable_collisions
pairs between the FT links and link5/link6/link_eef/gripper bodies.
Forward add_ft_sensor through the SRDF dispatch and expose it in
MoveItConfigsBuilder's URDF and SRDF xacro arg maps. Default true.

File: xarm_moveit_config/srdf/_xarm6_macro.srdf.xacro (robot description, xacro)
@@ -10,5 +10,6 @@
   <!-- SUBGROUPS: Groups can also be formed by referencing to already defined group names -->
   <xacro:macro name="xarm6_macro_srdf" params="prefix=''
-    add_gripper='false' add_vacuum_gripper='false' add_bio_gripper='false' add_other_geometry='false' ">
+    add_gripper='false' add_vacuum_gripper='false' add_bio_gripper='false' add_other_geometry='false'
+    add_ft_sensor='true' ">
     <group name="${prefix}xarm6">
       <joint name="${prefix}world_joint" />
@@ -19,4 +20,8 @@
       <joint name="${prefix}joint5" />
       <joint name="${prefix}joint6" />
+      <xacro:if value="${add_ft_sensor}">
+        <joint name="${prefix}joint_ft_adapter" />
+        <joint name="${prefix}joint_ft_sensor" />
+      </xacro:if>
       <joint name="${prefix}joint_eef" />
       <!-- To count in gripper TCP offset, if no need, please uncomment following 2 lines -->
@@ -202,4 +207,30 @@
     <disable_collisions link1="${prefix}link5" link2="${prefix}link6" reason="Adjacent" />
     <disable_collisions link1="${prefix}link6" link2="${prefix}link_eef" reason="Adjacent" />
+    <!-- FT sensor disable_collisions -->
+    <xacro:if value="${add_ft_sensor}">
+      <disable_collisions link1="${prefix}link5" link2="${prefix}link_ft_adapter" reason="Never" />
+      <disable_collisions link1="${prefix}link5" link2="${prefix}link_ft_sensor" reason="Never" />
+      <disable_collisions link1="${prefix}link6" link2="${prefix}link_ft_adapter" reason="Adjacent" />
+      <disable_collisions link1="${prefix}link6" link2="${prefix}link_ft_sensor" reason="Never" />
+      <disable_collisions link1="${prefix}link_ft_adapter" link2="${prefix}link_ft_sensor" reason="Adjacent" />
+      <disable_collisions link1="${prefix}link_ft_adapter" link2="${prefix}link_eef" reason="Never" />
+      <disable_collisions link1="${prefix}link_ft_sensor" link2="${prefix}link_eef" reason="Adjacent" />
+      <xacro:if value="${add_gripper}">
+        <disable_collisions link1="${prefix}link_ft_adapter" link2="${prefix}xarm_gripper_base_link" reason="Never" />
+        <disable_collisions link1="${prefix}link_ft_adapter" link2="${prefix}left_outer_knuckle" reason="Never" />
+        <disable_collisions link1="${prefix}link_ft_adapter" link2="${prefix}left_inner_knuckle" reason="Never" />
+        <disable_collisions link1="${prefix}link_ft_adapter" link2="${prefix}left_finger" reason="Never" />
+        <disable_collisions link1="${prefix}link_ft_adapter" link2="${prefix}right_outer_knuckle" reason="Never" />
+        <disable_collisions link1="${prefix}link_ft_adapter" link2="${prefix}right_inner_knuckle" reason="Never" />
+        <disable_collisions link1="${prefix}link_ft_adapter" link2="${prefix}right_finger" reason="Never" />
+        <disable_collisions link1="${prefix}link_ft_sensor" link2="${prefix}xarm_gripper_base_link" reason="Never" />
+        <disable_collisions link1="${prefix}link_ft_sensor" link2="${prefix}left_outer_knuckle" reason="Never" />
+        <disable_collisions link1="${prefix}link_ft_sensor" link2="${prefix}left_inner_knuckle" reason="Never" />
+        <disable_collisions link1="${prefix}link_ft_sensor" link2="${prefix}left_finger" reason="Never" />
+        <disable_collisions link1="${prefix}link_ft_sensor" link2="${prefix}right_outer_knuckle" reason="Never" />
+        <disable_collisions link1="${prefix}link_ft_sensor" link2="${prefix}right_inner_knuckle" reason="Never" />
+        <disable_collisions link1="${prefix}link_ft_sensor" link2="${prefix}right_finger" reason="Never" />
+      </xacro:if>
+    </xacro:if>
   </xacro:macro>
 </robot>

File: xarm_moveit_config/srdf/xarm.srdf.xacro (robot description, xacro)
@@ -9,6 +9,8 @@
   <xacro:arg name="add_bio_gripper" default="false" />
   <xacro:arg name="add_other_geometry" default="false" />
+  <xacro:arg name="add_ft_sensor" default="true" />
   <xacro:include filename="$(find xarm_moveit_config)/srdf/xarm_macro.srdf.xacro" />
   <xacro:xarm_macro_srdf prefix="$(arg prefix)" dof="$(arg dof)" robot_type="$(arg robot_type)"
-    add_gripper="$(arg add_gripper)" add_vacuum_gripper="$(arg add_vacuum_gripper)" add_bio_gripper="$(arg add_bio_gripper)" add_other_geometry="$(arg add_other_geometry)" />
+    add_gripper="$(arg add_gripper)" add_vacuum_gripper="$(arg add_vacuum_gripper)" add_bio_gripper="$(arg add_bio_gripper)" add_other_geometry="$(arg add_other_geometry)"
+    add_ft_sensor="$(arg add_ft_sensor)" />
 </robot>

File: xarm_moveit_config/srdf/xarm_macro.srdf.xacro (robot description, xacro)
@@ -2,5 +2,6 @@
 <robot xmlns:xacro="http://wiki.ros.org/xacro" name="xarm_srdf">
   <xacro:macro name="xarm_macro_srdf" params="prefix:='' dof:=7 robot_type:='xarm'
-    add_gripper:='false' add_vacuum_gripper:='false' add_bio_gripper:='false' add_other_geometry:='false' ">
+    add_gripper:='false' add_vacuum_gripper:='false' add_bio_gripper:='false' add_other_geometry:='false'
+    add_ft_sensor:='true' ">
     <xacro:if value="${dof == 5}">
       <xacro:include filename="$(find xarm_moveit_config)/srdf/_xarm5_macro.srdf.xacro" />
@@ -22,5 +23,6 @@
         <xacro:include filename="$(find xarm_moveit_config)/srdf/_xarm6_macro.srdf.xacro" />
         <xacro:xarm6_macro_srdf prefix="${prefix}"
-          add_gripper="${add_gripper}" add_vacuum_gripper="${add_vacuum_gripper}" add_bio_gripper="${add_bio_gripper}" add_other_geometry="${add_other_geometry}"  />
+          add_gripper="${add_gripper}" add_vacuum_gripper="${add_vacuum_gripper}" add_bio_gripper="${add_bio_gripper}" add_other_geometry="${add_other_geometry}"
+          add_ft_sensor="${add_ft_sensor}"  />
       </xacro:unless>
     </xacro:if>
