Commit message: Scale FT sensor mesh by 1e-3 for mm-to-m conversion
The exported STL uses millimetre-scale numeric values, which URDF
interprets as metres. Apply mesh scale="0.001 0.001 0.001" so the
sensor body renders at its real ~75 mm diameter instead of 75 m.
Replace common_link_visual/collision with raw mesh tags since the
helper macro doesn't accept a scale parameter.

File: xarm_description/urdf/ft_sensor/xarm_ft_sensor.urdf.xacro (robot description, xacro)
@@ -72,11 +72,18 @@
       </inertial>
       <xacro:if value="${use_mesh}">
-        <xacro:common_link_visual
-          mesh_filename="ft_sensor/xarm/visual/ft_sensor"
-          origin_xyz="0 0 -0.1191" origin_rpy="0 0 0"
-          material_name="${prefix}White"/>
-        <xacro:common_link_collision
-          mesh_filename="ft_sensor/xarm/collision/ft_sensor"
-          origin_xyz="0 0 -0.1191" origin_rpy="0 0 0"/>
+        <!-- STL units are millimetres; scale by 1e-3 to convert to URDF metres. -->
+        <visual>
+          <origin xyz="0 0 -0.1191" rpy="0 0 0"/>
+          <geometry>
+            <mesh filename="${mesh_path}/ft_sensor/xarm/visual/ft_sensor.${mesh_suffix}" scale="0.001 0.001 0.001"/>
+          </geometry>
+          <material name="${prefix}White"/>
+        </visual>
+        <collision>
+          <origin xyz="0 0 -0.1191" rpy="0 0 0"/>
+          <geometry>
+            <mesh filename="${mesh_path}/ft_sensor/xarm/collision/ft_sensor.${mesh_suffix}" scale="0.001 0.001 0.001"/>
+          </geometry>
+        </collision>
       </xacro:if>
       <xacro:unless value="${use_mesh}">

Commit message: Store FT sensor STL in metres
Rescale ft_sensor.stl vertices by 1e-3 in place so the mesh matches
the URDF convention of metre-scale STLs (~75 mm OD, ~58.6 mm tall).
Drop the scale="0.001 ..." attribute from the xacro and restore
common_link_visual/collision, consistent with the other xArm meshes.

File: xarm_description/urdf/ft_sensor/xarm_ft_sensor.urdf.xacro (robot description, xacro)
@@ -5,9 +5,10 @@
     Chain: attach_to -> link_ft_adapter (30 mm plate) -> link_ft_sensor (61 mm body).
     link_ft_sensor sits at the tool-output face; wrench values are referenced here.
-    Mesh note: the provided ft_sensor.stl contains the sensor body only (OD ~75 mm,
-    height ~58.6 mm). Its frame origin is offset: geometry sits at z in [60.5, 119.1] mm.
-    The visual origin below shifts it down by 119.1 mm so the top face lands at
-    link_ft_sensor origin (z=0) and the body extends in -Z back toward the adapter.
-    The mounting adapter has no mesh — rendered as a cylinder primitive.
+    Mesh note: ft_sensor.stl contains the sensor body only (OD ~75 mm, height
+    ~58.6 mm), stored in metres. Its frame origin is offset: geometry sits at
+    z in [0.0605, 0.1191] m. The visual origin below shifts it down by 0.1191 m
+    so the top face lands at link_ft_sensor origin (z=0) and the body extends
+    in -Z back toward the adapter. The mounting adapter has no mesh — rendered
+    as a cylinder primitive.
   -->
   <xacro:macro name="xarm_ft_sensor_urdf" params="
@@ -72,18 +73,11 @@
       </inertial>
       <xacro:if value="${use_mesh}">
-        <!-- STL units are millimetres; scale by 1e-3 to convert to URDF metres. -->
-        <visual>
-          <origin xyz="0 0 -0.1191" rpy="0 0 0"/>
-          <geometry>
-            <mesh filename="${mesh_path}/ft_sensor/xarm/visual/ft_sensor.${mesh_suffix}" scale="0.001 0.001 0.001"/>
-          </geometry>
-          <material name="${prefix}White"/>
-        </visual>
-        <collision>
-          <origin xyz="0 0 -0.1191" rpy="0 0 0"/>
-          <geometry>
-            <mesh filename="${mesh_path}/ft_sensor/xarm/collision/ft_sensor.${mesh_suffix}" scale="0.001 0.001 0.001"/>
-          </geometry>
-        </collision>
+        <xacro:common_link_visual
+          mesh_filename="ft_sensor/xarm/visual/ft_sensor"
+          origin_xyz="0 0 -0.1191" origin_rpy="0 0 0"
+          material_name="${prefix}White"/>
+        <xacro:common_link_collision
+          mesh_filename="ft_sensor/xarm/collision/ft_sensor"
+          origin_xyz="0 0 -0.1191" origin_rpy="0 0 0"/>
       </xacro:if>
       <xacro:unless value="${use_mesh}">
